Commit message: Finalize workspace urdf modelization

File: universal_robot/ur_description/urdf/env/box.urdf.xacro (robot description, xacro)
@@ -1,15 +1,25 @@
 <?xml version="1.0" ?>
 <robot xmlns:xacro="http://ros.org/wiki/xacro">
+<xacro:property name="half_pi" value="1.57079632679" />
+<!-- Definitions of box source dimensions  -->
+<xacro:property name="bsw" value="0.37" />
+<xacro:property name="bsh" value="0.245" />
+<xacro:property name="bsz" value="0.15" />
+<!-- Definitions of box destination dimensions  -->
+<xacro:property name="bdw" value="0.33" />
+<xacro:property name="bdh" value="0.255" />
+<xacro:property name="bdz" value="0.10" />
 <material name="white">
   <color rgba="1 1 1 0.7"/>
 </material>
 <material name="gray">
-  <color rgba="0.8 0.8 0.8 0.7"/>
+  <color rgba="0.8 0.8 0.0 0.7"/>
 </material>
 <xacro:macro name="box_source" params="name">
   <link name="${name}">
     <visual>
+      <origin rpy="0 0 ${half_pi}" xyz="-${bsh * 0.5} ${bsw * 0.5} -${bsz * 0.5}"/>
       <geometry>
-        <box size="0.38 0.25 0.15"/>
+        <box size="${bsw} ${bsh} ${bsz}"/>
       </geometry>
       <material name="white"/>
@@ -17,5 +27,6 @@
     <collision>
       <geometry>
-        <box size="0.38 0.25 0.05"/>
+      <!-- collision is smaller than the real size -->
+        <box size="${bsw} ${bsh} 0.05"/>
       </geometry>
     </collision>
@@ -25,6 +36,7 @@
   <link name="${name}">
     <visual>
+      <origin rpy="0 0 ${half_pi}" xyz="-${bdh * 0.5} ${bdw * 0.5} -${bdz * 0.5}"/>
       <geometry>
-        <box size="0.32 0.22 0.12"/>
+        <box size="${bdw} ${bdh} ${bdz}"/>
       </geometry>
       <material name="gray"/>
@@ -32,5 +44,5 @@
     <collision>
       <geometry>
-        <box size="0.32 0.22 0.12"/>
+        <box size="${bdw} ${bdh} ${bdz}"/>
       </geometry>
     </collision>

File: universal_robot/ur_description/urdf/project_environment.urdf.xacro (robot description, xacro)
@@ -2,22 +2,62 @@
 <robot xmlns:xacro="http://ros.org/wiki/xacro">
   <xacro:include filename="$(find ur_description)/urdf/env/box.urdf.xacro" />
+  <xacro:include filename="$(find ur_description)/urdf/env/table.urdf.xacro" />
+  <!-- Definitions of workspace dimensions (world) -->
+  <xacro:property name="ws_ysize" value="1.06" />
+  <xacro:property name="ws_xsize" value="1.19" />
   <link name="world"/>
   <xacro:table name="table"/>
   <xacro:box_source name="box_1"/>
+  <xacro:box_source name="box_2"/>
+  <xacro:box_source name="box_3"/>
+  <xacro:box_source name="box_4"/>
+  <xacro:box_source name="box_5"/>
+  <xacro:box_source name="box_6"/>
+  <xacro:box_source name="box_7"/>
   <xacro:box_destination name="box_dst"/>
   <joint name="world_table_link_joint" type="fixed">
     <parent link="world"/>
     <child link="table"/>
-    <origin xyz="0 0 0.05" rpy="0 0 0"/>
+    <origin xyz="-0.105 0.065 0.025" rpy="0 0 0"/>
   </joint>
   <joint name="world_box_1_joint" type="fixed">
     <parent link="world"/>
     <child link="box_1"/>
-    <origin xyz="2.0 0 0.0" rpy="0 0 0"/>
+    <origin xyz="0.0 ${ws_ysize - bsw} ${bsz}" rpy="0 0 0"/>
+  </joint>
+  <joint name="world_box_2_joint" type="fixed">
+    <parent link="world"/>
+    <child link="box_2"/>
+    <origin xyz="${-bsh*1} ${ws_ysize - bsw} ${bsz}" rpy="0 0 0"/>
+  </joint>
+  <joint name="world_box_3_joint" type="fixed">
+    <parent link="world"/>
+    <child link="box_3"/>
+    <origin xyz="${-bsh * 2} ${ws_ysize - bsw} ${bsz}" rpy="0 0 0"/>
+  </joint>
+  <joint name="world_box_4_joint" type="fixed">
+    <parent link="world"/>
+    <child link="box_4"/>
+    <origin xyz="${-bsh * 3 + bsh * 0.5} ${ws_ysize - bsw} ${bsz}" rpy="0 0 ${half_pi}"/>
+  </joint>
+  <joint name="world_box_5_joint" type="fixed">
+    <parent link="world"/>
+    <child link="box_5"/>
+    <origin xyz="${-bsh * 3 + bsh * 0.5} ${ws_ysize - bsw - bsh} ${bsz}" rpy="0 0 ${half_pi}"/>
+  </joint>
+  <joint name="world_box_6_joint" type="fixed">
+    <parent link="world"/>
+    <child link="box_6"/>
+    <origin xyz="${-bsh * 3 + bsh * 0.5} ${ws_ysize - bsw - bsh * 2} ${bsz}" rpy="0 0 ${half_pi}"/>
+  </joint>
+  <joint name="world_box_7_joint" type="fixed">
+    <parent link="world"/>
+    <child link="box_7"/>
+    <origin xyz="${-bsh * 3 + bsh * 0.5 + bsw} ${ws_ysize - bsw} ${bsz + tz}" rpy="0 0 ${half_pi}"/>
   </joint>
   <joint name="world_box_dst_joint" type="fixed">
     <parent link="world"/>
     <child link="box_dst"/>
-    <origin xyz="2.0 2.0 0.0" rpy="0 0 0"/>
+    <origin xyz="${-bsh * 3 + bsh * 0.5 - bsw} ${ws_ysize - bsw - bsh * 2} ${bdz}" rpy="0 0 0"/>
   </joint>
 </robot>

File: universal_robot/ur_description/urdf/ur5_joint_limited_robot.urdf.xacro (robot description, xacro)
@@ -20,5 +20,5 @@
     <parent link="table" />
     <child link = "base_link" />
-    <origin xyz="0.0 0.0 0.05" rpy="0.0 0.0 0.0" />
+    <origin xyz="-0.105 0.09 0.0" rpy="0.0 0.0 1.57079632679" />
   </joint>
 </robot>

File: universal_robot/ur_description/urdf/ur5_robot.urdf.xacro (robot description, xacro)
@@ -13,5 +13,5 @@
     <parent link="table" />
     <child link = "base_link" />
-    <origin xyz="0.0 0.0 0.0" rpy="0.0 0.0 0.0" />
+    <origin xyz="-0.105 0.09 0.0" rpy="0.0 0.0 1.57079632679" />
   </joint>
 </robot>

Commit message: Add suction pad and update starting script and move_group script

File: universal_robot/ur_description/urdf/env/box.urdf.xacro (robot description, xacro)
@@ -1,4 +1,4 @@
 <?xml version="1.0" ?>
-<robot xmlns:xacro="http://ros.org/wiki/xacro">
+<robot name="box" xmlns:xacro="http://ros.org/wiki/xacro">
 <xacro:property name="half_pi" value="1.57079632679" />
 <!-- Definitions of box source dimensions  -->

File: universal_robot/ur_description/urdf/env/table.urdf.xacro (robot description, xacro)
@@ -1,4 +1,4 @@
 <?xml version="1.0" ?>
-<robot xmlns:xacro="http://ros.org/wiki/xacro">
+<robot name="table" xmlns:xacro="http://ros.org/wiki/xacro">
 <!-- Definition of table dimensions  -->
 <xacro:property name="tw" value="0.5" />

File: universal_robot/ur_description/urdf/ur5_robot.urdf.xacro (robot description, xacro)
@@ -8,4 +8,6 @@
   <!-- ur5 -->
   <xacro:include filename="$(find ur_description)/urdf/ur5.urdf.xacro" />
+  <!-- actuator -->
+  <xacro:include filename="$(find ur_description)/urdf/actuator.urdf.xacro" />
   <!-- arm -->
   <xacro:ur5_robot prefix="" joint_limited="false"/>
@@ -15,3 +17,8 @@
     <origin xyz="-0.105 0.09 0.0" rpy="0.0 0.0 1.57079632679" />
   </joint>
+  <joint name="ee_link_table_base_plexi_joint" type="fixed">
+    <parent link="ee_link" />
+    <child link = "base_plexi" />
+    <origin xyz="0.0 0.0 0.0" rpy="0.0 1.57079632679 0.0" />
+  </joint>
 </robot>
