Commit message: Add walls and update working space

File: universal_robot/ur_description/urdf/env/table.urdf.xacro (robot description, xacro)
@@ -5,5 +5,5 @@
 <xacro:property name="th" value="0.515" />
 <xacro:property name="tz" value="0.025" />
-<material name="yellow">
+<material name="red">
   <color rgba="1 1 0 1"/>
 </material>

File: universal_robot/ur_description/urdf/project_environment.urdf.xacro (robot description, xacro)
@@ -3,4 +3,6 @@
   <xacro:include filename="$(find ur_description)/urdf/env/box.v2.urdf.xacro" />
   <xacro:include filename="$(find ur_description)/urdf/env/table.urdf.xacro" />
+  <xacro:include filename="$(find ur_description)/urdf/env/wall.urdf.xacro" />
+  <xacro:include filename="$(find ur_description)/urdf/env/camera.urdf.xacro" />
   <xacro:property name="half_pi" value="1.57079632679" />
   <!-- Definitions of workspace dimensions (world) -->
@@ -8,4 +10,8 @@
   <xacro:property name="ws_xsize" value="1.19" />
   <link name="world"/>
+  <xacro:generic_wall prefix="top" x="${wx}" y="${wdepth}" z="${wz}"/>
+  <xacro:generic_wall prefix="left" x="${wdepth}" y="${wy}" z="${wz}"/>
+  <xacro:generic_wall prefix="bottom" x="${wx}" y="${wdepth}" z="${wz}"/>
+  <xacro:generic_wall prefix="right" x="${wdepth}" y="${wy}" z="${wz}"/>
   <xacro:table name="table"/>
   <xacro:box_source name="box_1"/>
@@ -17,4 +23,29 @@
   <xacro:box_source name="box_7"/>
   <xacro:box_destination name="box_dst"/>
+  <joint name="world_top_wall_joint" type="fixed">
+    <parent link="world"/>
+    <child link="top_wall"/>
+    <origin xyz="0 ${wy} 0" rpy="0 0 0"/>
+  </joint>
+  <joint name="world_left_wall_joint" type="fixed">
+    <parent link="world"/>
+    <child link="left_wall"/>
+    <origin xyz="${wdepth} ${wy} 0" rpy="0 0 0"/>
+  </joint>
+  <joint name="world_bottom_wall_joint" type="fixed">
+    <parent link="world"/>
+    <child link="bottom_wall"/>
+    <origin xyz="0 -${wdepth + 0.05} 0" rpy="0 0 0"/>
+  </joint>
+  <joint name="world_right_wall_joint" type="fixed">
+    <parent link="world"/>
+    <child link="right_wall"/>
+    <origin xyz="-${wx} ${wy} 0" rpy="0 0 0"/>
+  </joint>
+  <joint name="world_camera_obstacle_joint" type="fixed">
+    <parent link="world"/>
+    <child link="camera_obstacle_link"/>
+    <origin xyz="-0.53 0.85 0.710" rpy="0 0 0"/>
+  </joint>
   <joint name="world_table_link_joint" type="fixed">
     <parent link="world"/>

File: universal_robot/ur_description/urdf/ur5_joint_limited_robot.urdf.xacro (robot description, xacro)
@@ -27,5 +27,5 @@
     <parent link="ee_link" />
     <child link = "base_plexi_link" />
-    <origin xyz="0.004 0.0 0.0 " rpy="1.57079632679 0.0 0.0" />
+    <origin xyz="0.004 0.0 0.0 " rpy="-1.57079632679 0.0 0.0" />
   </joint>
 </robot>

File: universal_robot/ur_description/urdf/ur5_robot.urdf.xacro (robot description, xacro)
@@ -21,5 +21,5 @@
     <parent link="ee_link" />
     <child link = "base_plexi_link" />
-    <origin xyz="0.004 0.0 0.0 " rpy="1.57079632679 0.0 0.0" />
+    <origin xyz="0.004 0.0 0.0 " rpy="1.57079632679 3.14159 0.0" />
   </joint>
 </robot>
