Commit message: Update automate program with joint state file reader

File: universal_robot/ur_description/urdf/env/wall.urdf.xacro (robot description, xacro)
@@ -5,5 +5,5 @@
 <xacro:property name="wz" value="1.1" />
 <material name="yellow">
-  <color rgba="1 1 0 0.25"/>
+  <color rgba="1 1 0 0.15"/>
 </material>
 <xacro:macro name="generic_wall" params="prefix x y z">
@@ -17,5 +17,5 @@
   </visual>
   <collision>
-    <!--<origin xyz="-${x / 2} -${y / 2} ${z / 2}" rpy="0 0 0"/>-->
+    <origin xyz="-${x / 2} -${y / 2} ${z / 2}" rpy="0 0 0"/>
     <geometry>
       <box size="${x} ${y} ${z}"/>

File: universal_robot/ur_description/urdf/project_environment.urdf.xacro (robot description, xacro)
@@ -6,23 +6,18 @@
   <xacro:include filename="$(find ur_description)/urdf/env/camera.urdf.xacro" />
   <xacro:property name="half_pi" value="1.57079632679" />
+  <xacro:property name="wall_delta" value="0.15" />
   <!-- Definitions of workspace dimensions (world) -->
   <link name="world"/>
-  <xacro:generic_wall prefix="top" x="${tx}" y="${wdepth}" z="${wz}"/>
-  <xacro:generic_wall prefix="left" x="${wdepth}" y="${ty}" z="${wz}"/>
-  <xacro:generic_wall prefix="bottom" x="${tx}" y="${wdepth}" z="${wz}"/>
-  <xacro:generic_wall prefix="right" x="${wdepth}" y="${ty}" z="${wz}"/>
+  <xacro:generic_wall prefix="top" x="${tx + wall_delta}" y="${wdepth}" z="${wz}"/>
+  <xacro:generic_wall prefix="left" x="${wdepth}" y="${ty + wall_delta}" z="${wz}"/>
+  <xacro:generic_wall prefix="bottom" x="${tx + wall_delta}" y="${wdepth}" z="${wz}"/>
+  <xacro:generic_wall prefix="right" x="${wdepth}" y="${ty + wall_delta}" z="${wz}"/>
   <xacro:table name="table"/>
   <xacro:box_source name="box_1"/>
-  <!--<xacro:box_source name="box_2"/>-->
-  <!--<xacro:box_source name="box_3"/>-->
-  <!--<xacro:box_source name="box_4"/>-->
-  <!--<xacro:box_source name="box_5"/>-->
-  <!--<xacro:box_source name="box_6"/>-->
-  <!--<xacro:box_source name="box_7"/>-->
   <xacro:box_destination name="box_dst"/>
   <joint name="world_top_wall_joint" type="fixed">
     <parent link="world"/>
     <child link="top_wall"/>
-    <origin xyz="0 ${ty} 0" rpy="0 0 0"/>
+    <origin xyz="${wall_delta} ${ty} 0" rpy="0 0 0"/>
   </joint>
   <joint name="world_left_wall_joint" type="fixed">
@@ -34,5 +29,5 @@
     <parent link="world"/>
     <child link="bottom_wall"/>
-    <origin xyz="0 -${0.15} 0" rpy="0 0 0"/>
+    <origin xyz="${wall_delta} -${wall_delta} 0" rpy="0 0 0"/>
     <!--<origin xyz="0.0 0.0 0.0" rpy="0 0 0"/>-->
   </joint>
@@ -40,6 +35,5 @@
     <parent link="world"/>
     <child link="right_wall"/>
-    <!--<origin xyz="-${tx} ${ty} 0" rpy="0 0 0"/>-->
-    <origin xyz="0.15 ${ty} 0" rpy="0 0 0"/>
+    <origin xyz="${wall_delta} ${ty} 0" rpy="0 0 0"/>
     <!--<origin xyz="0 -${0.15} 0" rpy="0 0 0"/>-->
   </joint>
@@ -59,39 +53,4 @@
     <origin xyz="-${0.4 + src_box_w / 2} ${0.5 + src_box_h / 2} 0.0" rpy="0 0 0"/>
   </joint>
-  <!--<joint name="world_box_1_joint" type="fixed">-->
-    <!--<parent link="world"/>-->
-    <!--<child link="box_1_base"/>-->
-    <!--<origin xyz="-${src_box_w * 0.5} ${ty - src_box_w * 0.5} 0.0" rpy="0 0 ${half_pi}"/>-->
-  <!--</joint>-->
-  <!--<joint name="world_box_2_joint" type="fixed">-->
-    <!--<parent link="world"/>-->
-    <!--<child link="box_2_base"/>-->
-    <!--<origin xyz="-${src_box_w * 0.5 + src_box_h * 1.0} ${ty - src_box_w * 0.5} 0.0" rpy="0 0 ${half_pi}"/>-->
-  <!--</joint>-->
-  <!--<joint name="world_box_3_joint" type="fixed">-->
-    <!--<parent link="world"/>-->
-    <!--<child link="box_3_base"/>-->
-    <!--<origin xyz="-${src_box_w * 0.5 + src_box_h * 2.25} ${ty - src_box_w * 0.5} 0.0" rpy="0 0 ${half_pi}"/>-->
-  <!--</joint>-->
-  <!--<joint name="world_box_4_joint" type="fixed">-->
-    <!--<parent link="world"/>-->
-    <!--<child link="box_4_base"/>-->
-    <!--<origin xyz="-${src_box_w * 0.5 + src_box_h * 2.5} ${ty - src_box_w - src_box_h * 0.5} 0.0" rpy="0 0 0"/>-->
-  <!--</joint>-->
-  <!--<joint name="world_box_5_joint" type="fixed">-->
-    <!--<parent link="world"/>-->
-    <!--<child link="box_5_base"/>-->
-    <!--<origin xyz="-${src_box_w * 0.5 + src_box_h * 2.5} ${ty - src_box_w - src_box_h * 1.5} 0.0" rpy="0 0 0"/>-->
-  <!--</joint>-->
-  <!--<joint name="world_box_6_joint" type="fixed">-->
-    <!--<parent link="world"/>-->
-    <!--<child link="box_6_base"/>-->
-    <!--<origin xyz="-${src_box_w * 0.5 + src_box_h * 2.5} ${ty - src_box_w - src_box_h * 2.5} 0.0" rpy="0 0 0"/>-->
-  <!--</joint>-->
-  <!--<joint name="world_box_7_joint" type="fixed">-->
-    <!--<parent link="world"/>-->
-    <!--<child link="box_7_base"/>-->
-    <!--<origin xyz="${src_box_w * 0.5 - src_box_h * 2.5} ${ty - src_box_w - src_box_h * 0.5} ${tz}" rpy="0 0 0"/>-->
-  <!--</joint>-->
   <joint name="world_box_dst_joint" type="fixed">
     <parent link="world"/>

File: universal_robot/ur_description/urdf/ur5_joint_limited_robot.urdf.xacro (robot description, xacro)
@@ -22,5 +22,5 @@
     <parent link="table" />
     <child link = "base_link" />
-    <origin xyz="-0.125 0.125 0.0" rpy="0.0 0.0 ${pi / 4.0}" />
+    <origin xyz="-0.125 0.125 0.001" rpy="0.0 0.0 ${pi / 4.0}" />
   </joint>
   <joint name="ee_joint" type="fixed">

File: universal_robot/ur_description/urdf/ur5_robot.urdf.xacro (robot description, xacro)
@@ -16,5 +16,5 @@
     <parent link="table" />
     <child link = "base_link" />
-    <origin xyz="-0.125 0.125 0.0" rpy="0.0 0.0 0.7853981633974483" />
+    <origin xyz="-0.125 0.125 0.001" rpy="0.0 0.0 0.7853981633974483" />
   </joint>
   <joint name="ee_joint" type="fixed">
