Commit message: Update code to display tf, replan etc

File: universal_robot/ur_description/urdf/env/camera.urdf.xacro (robot description, xacro)
@@ -2,7 +2,7 @@
 <robot name="wall" xmlns:xacro="http://ros.org/wiki/xacro">
 <!-- Definition of table dimensions  -->
-<xacro:property name="cam_x" value="0.27" />
-<xacro:property name="cam_y" value="0.05" />
-<xacro:property name="cam_z" value="0.07" />
+<xacro:property name="cam_x" value="0.30" />
+<xacro:property name="cam_y" value="0.07" />
+<xacro:property name="cam_z" value="0.10" />
 <material name="black">
   <color rgba="0 0 0 0.8"/>

File: universal_robot/ur_description/urdf/env/wall.urdf.xacro (robot description, xacro)
@@ -7,5 +7,5 @@
 <xacro:property name="wz" value="1.06" />
 <material name="yellow">
-  <color rgba="1 1 0 0.5"/>
+  <color rgba="1 1 0 0.25"/>
 </material>
 <xacro:macro name="generic_wall" params="prefix x y z">

File: universal_robot/ur_description/urdf/project_environment.urdf.xacro (robot description, xacro)
@@ -66,5 +66,5 @@
     <parent link="world"/>
     <child link="box_3_base"/>
-    <origin xyz="-${src_box_w * 0.5 + src_box_h * 2.0} ${ws_ysize - src_box_w * 0.5} 0.0" rpy="0 0 ${half_pi}"/>
+    <origin xyz="-${src_box_w * 0.5 + src_box_h * 2.25} ${ws_ysize - src_box_w * 0.5} 0.0" rpy="0 0 ${half_pi}"/>
   </joint>
   <joint name="world_box_4_joint" type="fixed">

Commit message: update intrinsec and extrinsec parameter

File: universal_robot/ur_description/urdf/env/camera.urdf.xacro (robot description, xacro)
@@ -2,5 +2,5 @@
 <robot name="wall" xmlns:xacro="http://ros.org/wiki/xacro">
 <!-- Definition of camera dimensions  -->
-<xacro:property name="cam_x" value="0.30" />
+<xacro:property name="cam_x" value="0.40" />
 <xacro:property name="cam_y" value="0.07" />
 <xacro:property name="cam_z" value="0.10" />
