Commit message: Update the environment urdf: box -> v2

File: universal_robot/ur_description/urdf/env/box.v2.urdf.xacro (robot description, xacro)
@@ -1,103 +1,125 @@
 ﻿<?xml version="1.0" encoding="UTF-8"?>
-<robot name="box">
-  <link name="base">
-    <visual>
-      <origin xyz="0 0 0" rpy="0 0 0"/>
-      <geometry>
-        <box size="0.37 0.245 .01"/>
-      </geometry>
-      <material name="mat1">
-        <color rgba="1 1 1 1"/>
-      </material>
-    </visual>
-    <collision>
-      <geometry>
-        <box size="0.37 0.245 .01"/>
-      </geometry>
-    </collision>
-  </link>
-  <link name="left">
-    <visual>
-      <origin xyz="0 0 0" rpy="0 0 0"/>
-      <geometry>
-        <box size="0.37 0.01 .15"/>
-      </geometry>
-      <material name="mat2">
-        <color rgba="1 0 1 1"/>
-      </material>
-    </visual>
-    <collision>
-      <geometry>
-        <box size="0.37 0.01 .15"/>
-      </geometry>
-    </collision>
-  </link>
-  <link name="right">
-    <visual>
-      <origin xyz="0 0 0" rpy="0 0 0"/>
-      <geometry>
-        <box size="0.37 0.01 .15"/>
-      </geometry>
-      <material name="mat3">
-        <color rgba="1 1 0 1"/>
-      </material>
-    </visual>
-    <collision>
-      <geometry>
-        <box size="0.37 0.01 .15"/>
-      </geometry>
-    </collision>
-  </link>
-  <link name="top">
-    <visual>
-      <origin xyz="0 0 0" rpy="0 0 0"/>
-      <geometry>
-        <box size="0.01 0.245 .15"/>
-      </geometry>
-      <material name="mat4">
-        <color rgba="0 1 1 1"/>
-      </material>
-    </visual>
-    <collision>
-      <geometry>
-        <box size="0.01 0.245 .15"/>
-      </geometry>
-    </collision>
-  </link>
-  <link name="bottom">
-    <visual>
-      <origin xyz="0 0 0" rpy="0 0 0"/>
-      <geometry>
-        <box size="0.01 0.245 .15"/>
-      </geometry>
-      <material name="mat5">
-        <color rgba="0 0 1 1"/>
-      </material>
-    </visual>
-    <collision>
-      <geometry>
-        <box size="0.01 0.245 .15"/>
-      </geometry>
-    </collision>
-  </link>
-  <joint name="base_to_left" type="fixed">
-    <parent link="base"/>
-    <child link="left"/>
-    <origin xyz="0 -0.122 0.075 "/>
-  </joint>
-  <joint name="base_to_right" type="fixed">
-    <parent link="base"/>
-    <child link="right"/>
-    <origin xyz="0 0.122 0.075 "/>
-  </joint>
-  <joint name="base_to_top" type="fixed">
-    <parent link="base"/>
-    <child link="top"/>
-    <origin xyz="0.185 0.0 0.075 "/>
-  </joint>
-  <joint name="base_to_bottom" type="fixed">
-    <parent link="base"/>
-    <child link="bottom"/>
-    <origin xyz="-0.185 0.0 0.075 "/>
-  </joint>
+<robot name="box" xmlns:xacro="http://ros.org/wiki/xacro">
+  <!-- Box plastic depth -->
+  <xacro:property name="box_side_depth" value="0.01" />
+  <!-- Definitions of box source dimensions  -->
+  <xacro:property name="src_box_w" value="0.37" />
+  <xacro:property name="src_box_h" value="0.245" />
+  <xacro:property name="src_box_z" value="0.15" />
+  <!-- Definitions of box destination dimensions  -->
+  <xacro:property name="dst_box_w" value="0.33" />
+  <xacro:property name="dst_box_h" value="0.255" />
+  <xacro:property name="dst_box_z" value="0.10" />
+  <material name="bscolor">
+    <color rgba="1 1 1 0.85"/>
+  </material>
+  <xacro:macro name="generic_box"
+    params="prefix bsw bsh bsz depth">
+    <link name="${prefix}_base">
+      <visual>
+        <origin xyz="0 0 0" rpy="0 0 0"/>
+        <geometry>
+          <box size="${bsw} ${bsh} ${depth}"/>
+        </geometry>
+        <material name="bscolor" />
+      </visual>
+      <collision>
+        <geometry>
+          <box size="${bsw} ${bsh} ${depth}"/>
+        </geometry>
+      </collision>
+    </link>
+    <link name="${prefix}_left">
+      <visual>
+        <origin xyz="0 0 0" rpy="0 0 0"/>
+        <geometry>
+          <box size="${bsw} ${depth} ${bsz}"/>
+        </geometry>
+        <material name="bscolor" />
+      </visual>
+      <collision>
+        <geometry>
+          <box size="${bsw} ${depth} ${bsz}"/>
+        </geometry>
+      </collision>
+    </link>
+    <link name="${prefix}_right">
+      <visual>
+        <origin xyz="0 0 0" rpy="0 0 0"/>
+        <geometry>
+          <box size="${bsw} ${depth} ${bsz}"/>
+        </geometry>
+        <material name="bscolor" />
+      </visual>
+      <collision>
+        <geometry>
+          <box size="${bsw} ${depth} ${bsz}"/>
+        </geometry>
+      </collision>
+    </link>
+    <link name="${prefix}_top">
+      <visual>
+        <origin xyz="0 0 0" rpy="0 0 0"/>
+        <geometry>
+          <box size="${depth} ${bsh} ${bsz}"/>
+        </geometry>
+        <material name="bscolor" />
+      </visual>
+      <collision>
+        <geometry>
+          <box size="${depth} ${bsh} ${bsz}"/>
+        </geometry>
+      </collision>
+    </link>
+    <link name="${prefix}_bottom">
+      <visual>
+        <origin xyz="0 0 0" rpy="0 0 0"/>
+        <geometry>
+          <box size="${depth} ${bsh} ${bsz}"/>
+        </geometry>
+        <material name="bscolor" />
+      </visual>
+      <collision>
+        <geometry>
+          <box size="${depth} ${bsh} ${bsz}"/>
+        </geometry>
+      </collision>
+    </link>
+    <joint name="${prefix}_base_to_left" type="fixed">
+      <parent link="${prefix}_base"/>
+      <child link="${prefix}_left"/>
+      <origin xyz="0.0 -${bsh * 0.5 - depth * 0.5} ${bsz * 0.5 - depth * 0.5}"/>
+    </joint>
+    <joint name="${prefix}_base_to_right" type="fixed">
+      <parent link="${prefix}_base"/>
+      <child link="${prefix}_right"/>
+      <origin xyz="0.0 ${bsh * 0.5 - depth * 0.5} ${bsz * 0.5 - depth * 0.5}"/>
+    </joint>
+    <joint name="${prefix}_base_to_top" type="fixed">
+      <parent link="${prefix}_base"/>
+      <child link="${prefix}_top"/>
+      <origin xyz="${bsw * 0.5 - depth * 0.5} 0.0 ${bsz * 0.5 - depth * 0.5}"/>
+    </joint>
+    <joint name="${prefix}_base_to_bottom" type="fixed">
+      <parent link="${prefix}_base"/>
+      <child link="${prefix}_bottom"/>
+      <origin xyz="-${bsw * 0.5 - depth * 0.5} 0.0 ${bsz * 0.5 - depth * 0.5}"/>
+    </joint>
+  </xacro:macro>
+  <xacro:macro name="box_source" params="name">
+    <xacro:generic_box
+      prefix="${name}"
+      bsw="${src_box_w}"
+      bsh="${src_box_h}"
+      bsz="${src_box_z}"
+      depth="${box_side_depth}"/>
+  </xacro:macro>
+  <xacro:macro name="box_destination" params="name">
+    <xacro:generic_box
+      prefix="${name}"
+      bsw="${dst_box_w}"
+      bsh="${dst_box_h}"
+      bsz="${dst_box_z}"
+      depth="${box_side_depth}"/>
+  </xacro:macro>
 </robot>

File: universal_robot/ur_description/urdf/project_environment.urdf.xacro (robot description, xacro)
@@ -1,6 +1,7 @@
 <?xml version="1.0" ?>
 <robot xmlns:xacro="http://ros.org/wiki/xacro">
-  <xacro:include filename="$(find ur_description)/urdf/env/box.urdf.xacro" />
+  <xacro:include filename="$(find ur_description)/urdf/env/box.v2.urdf.xacro" />
   <xacro:include filename="$(find ur_description)/urdf/env/table.urdf.xacro" />
+  <xacro:property name="half_pi" value="1.57079632679" />
   <!-- Definitions of workspace dimensions (world) -->
   <xacro:property name="ws_ysize" value="1.06" />
@@ -8,5 +9,5 @@
   <link name="world"/>
   <xacro:table name="table"/>
-  <!--<xacro:box_source name="box_1"/>-->
+  <xacro:box_source name="box_1"/>
   <xacro:box_source name="box_2"/>
   <xacro:box_source name="box_3"/>
@@ -21,43 +22,43 @@
     <origin xyz="-0.105 0.065 0.025" rpy="0 0 0"/>
   </joint>
-  <!--<joint name="world_box_1_joint" type="fixed">-->
-    <!--<parent link="world"/>-->
-    <!--<child link="box_1"/>-->
-    <!--<origin xyz="0.0 ${ws_ysize - bsw} ${bsz}" rpy="0 0 0"/>-->
-  <!--</joint>-->
+  <joint name="world_box_1_joint" type="fixed">
+    <parent link="world"/>
+    <child link="box_1_base"/>
+    <origin xyz="-${src_box_w * 0.5} ${ws_ysize - src_box_w * 0.5} 0.0" rpy="0 0 ${half_pi}"/>
+  </joint>
   <joint name="world_box_2_joint" type="fixed">
     <parent link="world"/>
-    <child link="box_2"/>
-    <origin xyz="${-bsh*1} ${ws_ysize - bsw} ${bsz}" rpy="0 0 0"/>
+    <child link="box_2_base"/>
+    <origin xyz="-${src_box_w * 0.5 + src_box_h * 1.0} ${ws_ysize - src_box_w * 0.5} 0.0" rpy="0 0 ${half_pi}"/>
   </joint>
   <joint name="world_box_3_joint" type="fixed">
     <parent link="world"/>
-    <child link="box_3"/>
-    <origin xyz="${-bsh * 2} ${ws_ysize - bsw} ${bsz}" rpy="0 0 0"/>
+    <child link="box_3_base"/>
+    <origin xyz="-${src_box_w * 0.5 + src_box_h * 2.0} ${ws_ysize - src_box_w * 0.5} 0.0" rpy="0 0 ${half_pi}"/>
   </joint>
   <joint name="world_box_4_joint" type="fixed">
     <parent link="world"/>
-    <child link="box_4"/>
-    <origin xyz="${-bsh * 3 + bsh * 0.5} ${ws_ysize - bsw} ${bsz}" rpy="0 0 ${half_pi}"/>
+    <child link="box_4_base"/>
+    <origin xyz="-${src_box_w * 0.5 + src_box_h * 2.5} ${ws_ysize - src_box_w - src_box_h * 0.5} 0.0" rpy="0 0 0"/>
   </joint>
   <joint name="world_box_5_joint" type="fixed">
     <parent link="world"/>
-    <child link="box_5"/>
-    <origin xyz="${-bsh * 3 + bsh * 0.5} ${ws_ysize - bsw - bsh} ${bsz}" rpy="0 0 ${half_pi}"/>
+    <child link="box_5_base"/>
+    <origin xyz="-${src_box_w * 0.5 + src_box_h * 2.5} ${ws_ysize - src_box_w - src_box_h * 1.5} 0.0" rpy="0 0 0"/>
   </joint>
   <joint name="world_box_6_joint" type="fixed">
     <parent link="world"/>
-    <child link="box_6"/>
-    <origin xyz="${-bsh * 3 + bsh * 0.5} ${ws_ysize - bsw - bsh * 2} ${bsz}" rpy="0 0 ${half_pi}"/>
+    <child link="box_6_base"/>
+    <origin xyz="-${src_box_w * 0.5 + src_box_h * 2.5} ${ws_ysize - src_box_w - src_box_h * 2.5} 0.0" rpy="0 0 0"/>
   </joint>
   <joint name="world_box_7_joint" type="fixed">
     <parent link="world"/>
-    <child link="box_7"/>
-    <origin xyz="${-bsh * 3 + bsh * 0.5 + bsw} ${ws_ysize - bsw} ${bsz + tz}" rpy="0 0 ${half_pi}"/>
+    <child link="box_7_base"/>
+    <origin xyz="${src_box_w * 0.5 - src_box_h * 2.5} ${ws_ysize - src_box_w - src_box_h * 0.5} ${tz}" rpy="0 0 0"/>
   </joint>
   <joint name="world_box_dst_joint" type="fixed">
     <parent link="world"/>
-    <child link="box_dst"/>
-    <origin xyz="${-bsh * 3 + bsh * 0.5 - bsw} ${ws_ysize - bsw - bsh * 2} ${bdz}" rpy="0 0 0"/>
+    <child link="box_dst_base"/>
+    <origin xyz="-${src_box_w * 1.0 + dst_box_h * 0.5 + src_box_h * 2.5} ${ws_ysize - src_box_w - src_box_h * 2.0 + dst_box_h * 0.5} 0.0" rpy="0 0 ${half_pi}"/>
   </joint>
 </robot>

Commit message: Update URDF to new workcell

File: universal_robot/ur_description/urdf/env/box.v2.urdf.xacro (robot description, xacro)
@@ -4,7 +4,7 @@
   <xacro:property name="box_side_depth" value="0.01" />
   <!-- Definitions of box source dimensions  -->
-  <xacro:property name="src_box_w" value="0.37" />
-  <xacro:property name="src_box_h" value="0.245" />
-  <xacro:property name="src_box_z" value="0.15" />
+  <xacro:property name="src_box_w" value="0.43" />
+  <xacro:property name="src_box_h" value="0.28" />
+  <xacro:property name="src_box_z" value="0.164" />
   <!-- Definitions of box destination dimensions  -->
   <xacro:property name="dst_box_w" value="0.33" />

File: universal_robot/ur_description/urdf/env/camera.urdf.xacro (robot description, xacro)
@@ -1,14 +1,23 @@
 <?xml version="1.0" ?>
 <robot name="wall" xmlns:xacro="http://ros.org/wiki/xacro">
-<!-- Definition of table dimensions  -->
+<!-- Definition of camera dimensions  -->
 <xacro:property name="cam_x" value="0.30" />
 <xacro:property name="cam_y" value="0.07" />
 <xacro:property name="cam_z" value="0.10" />
+<!-- Definition of camera dimensions  -->
+<xacro:property name="hor_bulk_x" value="0.09" />
+<xacro:property name="hor_bulk_y" value="0.563" />
+<xacro:property name="hor_bulk_z" value="0.045" />
+<xacro:property name="vert_bulk_x" value="0.09" />
+<xacro:property name="vert_bulk_y" value="0.045" />
+<xacro:property name="vert_bulk_z" value="0.965" />
 <material name="black">
   <color rgba="0 0 0 0.8"/>
 </material>
+<material name="gray">
+  <color rgba="0.4 0.4 0.4 0.8"/>
+</material>
 <link name="camera_obstacle_link">
   <visual>
-    <origin xyz="-${cam_x / 2} ${cam_y / 2} ${cam_z / 2}" rpy="0 0 0"/>
     <geometry>
       <box size="${cam_x} ${cam_y} ${cam_z}"/>
@@ -17,5 +26,4 @@
   </visual>
   <collision>
-    <origin xyz="-${cam_x / 2} ${cam_y / 2} ${cam_z / 2}" rpy="0 0 0"/>
     <geometry>
       <box size="${cam_x} ${cam_y} ${cam_z}"/>
@@ -23,3 +31,43 @@
   </collision>
 </link>
+<link name="camera_hor_fixation_obstacle_link">
+  <visual>
+    <origin xyz="-${hor_bulk_x / 2} ${hor_bulk_y / 2} ${hor_bulk_z / 2}" rpy="0 0 0"/>
+    <geometry>
+      <box size="${hor_bulk_x} ${hor_bulk_y} ${hor_bulk_z}"/>
+    </geometry>
+    <material name="gray" />
+  </visual>
+  <collision>
+    <origin xyz="-${hor_bulk_x / 2} ${hor_bulk_y / 2} ${hor_bulk_z / 2}" rpy="0 0 0"/>
+    <geometry>
+      <box size="${hor_bulk_x} ${hor_bulk_y} ${hor_bulk_z}"/>
+    </geometry>
+  </collision>
+</link>
+<link name="camera_vert_fixation_obstacle_link">
+  <visual>
+    <origin xyz="-${vert_bulk_x / 2} ${vert_bulk_y / 2} ${vert_bulk_z / 2}" rpy="0 0 0"/>
+    <geometry>
+      <box size="${vert_bulk_x} ${vert_bulk_y} ${vert_bulk_z}"/>
+    </geometry>
+    <material name="gray" />
+  </visual>
+  <collision>
+    <origin xyz="-${vert_bulk_x / 2} ${vert_bulk_y / 2} ${vert_bulk_z / 2}" rpy="0 0 0"/>
+    <geometry>
+      <box size="${vert_bulk_x} ${vert_bulk_y} ${vert_bulk_z}"/>
+    </geometry>
+  </collision>
+</link>
+<joint name="camera_vert_hor_joint" type="fixed">
+  <parent link="camera_vert_fixation_obstacle_link"/>
+  <child link="camera_hor_fixation_obstacle_link"/>
+  <origin xyz="0.0 -${hor_bulk_y} ${vert_bulk_z - hor_bulk_z}" rpy="0 0 0"/>
+</joint>
+<joint name="camera_hor_joint" type="fixed">
+  <parent link="camera_hor_fixation_obstacle_link"/>
+  <child link="camera_obstacle_link"/>
+  <origin xyz="-${hor_bulk_x / 2} 0.16 -0.044" rpy="0 0 0"/>
+</joint>
 </robot>

File: universal_robot/ur_description/urdf/env/table.urdf.xacro (robot description, xacro)
@@ -2,22 +2,24 @@
 <robot name="table" xmlns:xacro="http://ros.org/wiki/xacro">
 <!-- Definition of table dimensions  -->
-<xacro:property name="tw" value="0.5" />
-<xacro:property name="th" value="0.515" />
-<xacro:property name="tz" value="0.025" />
-<material name="red">
-  <color rgba="1 1 0 1"/>
+<xacro:property name="tx" value="1.20" />
+<xacro:property name="ty" value="1.0" />
+<xacro:property name="tz" value="0.56" />
+<material name="white">
+  <color rgba="0.85 0.85 0.85 1"/>
 </material>
 <xacro:macro name="table" params="name">
   <link name="table">
     <visual>
-      <!-- xyz point is zero of the parent link -->
-      <origin rpy="0 0 0" xyz="-${tw * 0.5} ${th * 0.5} -${tz * 0.5}"/>
+      <!-- xyz point is zero of tye parent link -->
+      <origin rpy="0 0 0" xyz="-${tx * 0.5} ${ty * 0.5} -${tz * 0.5}"/>
       <geometry>
-        <box size="${tw} ${th} ${tz}"/>
+        <box size="${tx} ${ty} ${tz}"/>
       </geometry>
+      <material name="white" />
     </visual>
     <collision>
+      <origin rpy="0 0 0" xyz="-${tx * 0.5} ${ty * 0.5} -${tz * 0.5}"/>
       <geometry>
-        <box size="${tw} ${th} ${tz}"/>
+        <box size="${tx} ${ty} ${tz}"/>
       </geometry>
     </collision>

File: universal_robot/ur_description/urdf/env/wall.urdf.xacro (robot description, xacro)
@@ -2,8 +2,6 @@
 <robot name="wall" xmlns:xacro="http://ros.org/wiki/xacro">
 <!-- Definition of table dimensions  -->
-<xacro:property name="wx" value="1.18" />
-<xacro:property name="wy" value="1.08" />
 <xacro:property name="wdepth" value="0.02" />
-<xacro:property name="wz" value="1.06" />
+<xacro:property name="wz" value="1.1" />
 <material name="yellow">
   <color rgba="1 1 0 0.25"/>
@@ -19,5 +17,5 @@
   </visual>
   <collision>
-    <origin xyz="-${x / 2} -${y / 2} ${z / 2}" rpy="0 0 0"/>
+    <!--<origin xyz="-${x / 2} -${y / 2} ${z / 2}" rpy="0 0 0"/>-->
     <geometry>
       <box size="${x} ${y} ${z}"/>

File: universal_robot/ur_description/urdf/project_environment.urdf.xacro (robot description, xacro)
@@ -7,11 +7,9 @@
   <xacro:property name="half_pi" value="1.57079632679" />
   <!-- Definitions of workspace dimensions (world) -->
-  <xacro:property name="ws_ysize" value="1.06" />
-  <xacro:property name="ws_xsize" value="1.19" />
   <link name="world"/>
-  <xacro:generic_wall prefix="top" x="${wx}" y="${wdepth}" z="${wz}"/>
-  <xacro:generic_wall prefix="left" x="${wdepth}" y="${wy}" z="${wz}"/>
-  <xacro:generic_wall prefix="bottom" x="${wx}" y="${wdepth}" z="${wz}"/>
-  <xacro:generic_wall prefix="right" x="${wdepth}" y="${wy}" z="${wz}"/>
+  <xacro:generic_wall prefix="top" x="${tx}" y="${wdepth}" z="${wz}"/>
+  <xacro:generic_wall prefix="left" x="${wdepth}" y="${ty}" z="${wz}"/>
+  <xacro:generic_wall prefix="bottom" x="${tx}" y="${wdepth}" z="${wz}"/>
+  <xacro:generic_wall prefix="right" x="${wdepth}" y="${ty}" z="${wz}"/>
   <xacro:table name="table"/>
   <xacro:box_source name="box_1"/>
@@ -26,75 +24,78 @@
     <parent link="world"/>
     <child link="top_wall"/>
-    <origin xyz="0 ${wy} 0" rpy="0 0 0"/>
+    <origin xyz="0 ${ty} 0" rpy="0 0 0"/>
   </joint>
   <joint name="world_left_wall_joint" type="fixed">
     <parent link="world"/>
     <child link="left_wall"/>
-    <origin xyz="${wdepth} ${wy} 0" rpy="0 0 0"/>
+    <origin xyz="-${tx + wdepth} ${ty} 0" rpy="0 0 0"/>
   </joint>
   <joint name="world_bottom_wall_joint" type="fixed">
     <parent link="world"/>
     <child link="bottom_wall"/>
-    <origin xyz="0 -${wdepth + 0.30} 0" rpy="0 0 0"/>
+    <origin xyz="0 -${0.15} 0" rpy="0 0 0"/>
+    <!--<origin xyz="0.0 0.0 0.0" rpy="0 0 0"/>-->
   </joint>
   <joint name="world_right_wall_joint" type="fixed">
     <parent link="world"/>
     <child link="right_wall"/>
-    <origin xyz="-${wx} ${wy} 0" rpy="0 0 0"/>
+    <!--<origin xyz="-${tx} ${ty} 0" rpy="0 0 0"/>-->
+    <origin xyz="0.15 ${ty} 0" rpy="0 0 0"/>
+    <!--<origin xyz="0 -${0.15} 0" rpy="0 0 0"/>-->
   </joint>
   <joint name="world_camera_obstacle_joint" type="fixed">
     <parent link="world"/>
-    <child link="camera_obstacle_link"/>
-    <origin xyz="-0.234 0.555 0.90" rpy="0 0 0"/>
+    <child link="camera_vert_fixation_obstacle_link"/>
+    <origin xyz="-0.553 ${ty} 0.0" rpy="0 0 0"/>
   </joint>
   <joint name="world_table_link_joint" type="fixed">
     <parent link="world"/>
     <child link="table"/>
-    <origin xyz="-0.105 0.065 0.025" rpy="0 0 0"/>
+    <origin xyz="-0.0 0.0 0.0" rpy="0 0 0"/>
   </joint>
   <joint name="world_box_1_joint" type="fixed">
     <parent link="world"/>
     <child link="box_1_base"/>
-    <origin xyz="-${src_box_w * 0.5 + 0.2253} ${ws_ysize - src_box_h * 0.25 - 0.375} ${tz}" rpy="0 0 0"/>
+    <origin xyz="-${0.4 + src_box_w / 2} ${0.5 + src_box_h / 2} 0.0" rpy="0 0 0"/>
   </joint>
   <!--<joint name="world_box_1_joint" type="fixed">-->
     <!--<parent link="world"/>-->
     <!--<child link="box_1_base"/>-->
-    <!--<origin xyz="-${src_box_w * 0.5} ${ws_ysize - src_box_w * 0.5} 0.0" rpy="0 0 ${half_pi}"/>-->
+    <!--<origin xyz="-${src_box_w * 0.5} ${ty - src_box_w * 0.5} 0.0" rpy="0 0 ${half_pi}"/>-->
   <!--</joint>-->
   <!--<joint name="world_box_2_joint" type="fixed">-->
     <!--<parent link="world"/>-->
     <!--<child link="box_2_base"/>-->
-    <!--<origin xyz="-${src_box_w * 0.5 + src_box_h * 1.0} ${ws_ysize - src_box_w * 0.5} 0.0" rpy="0 0 ${half_pi}"/>-->
+    <!--<origin xyz="-${src_box_w * 0.5 + src_box_h * 1.0} ${ty - src_box_w * 0.5} 0.0" rpy="0 0 ${half_pi}"/>-->
   <!--</joint>-->
   <!--<joint name="world_box_3_joint" type="fixed">-->
     <!--<parent link="world"/>-->
     <!--<child link="box_3_base"/>-->
-    <!--<origin xyz="-${src_box_w * 0.5 + src_box_h * 2.25} ${ws_ysize - src_box_w * 0.5} 0.0" rpy="0 0 ${half_pi}"/>-->
+    <!--<origin xyz="-${src_box_w * 0.5 + src_box_h * 2.25} ${ty - src_box_w * 0.5} 0.0" rpy="0 0 ${half_pi}"/>-->
   <!--</joint>-->
   <!--<joint name="world_box_4_joint" type="fixed">-->
     <!--<parent link="world"/>-->
     <!--<child link="box_4_base"/>-->
-    <!--<origin xyz="-${src_box_w * 0.5 + src_box_h * 2.5} ${ws_ysize - src_box_w - src_box_h * 0.5} 0.0" rpy="0 0 0"/>-->
+    <!--<origin xyz="-${src_box_w * 0.5 + src_box_h * 2.5} ${ty - src_box_w - src_box_h * 0.5} 0.0" rpy="0 0 0"/>-->
   <!--</joint>-->
   <!--<joint name="world_box_5_joint" type="fixed">-->
     <!--<parent link="world"/>-->
     <!--<child link="box_5_base"/>-->
-    <!--<origin xyz="-${src_box_w * 0.5 + src_box_h * 2.5} ${ws_ysize - src_box_w - src_box_h * 1.5} 0.0" rpy="0 0 0"/>-->
+    <!--<origin xyz="-${src_box_w * 0.5 + src_box_h * 2.5} ${ty - src_box_w - src_box_h * 1.5} 0.0" rpy="0 0 0"/>-->
   <!--</joint>-->
   <!--<joint name="world_box_6_joint" type="fixed">-->
     <!--<parent link="world"/>-->
     <!--<child link="box_6_base"/>-->
-    <!--<origin xyz="-${src_box_w * 0.5 + src_box_h * 2.5} ${ws_ysize - src_box_w - src_box_h * 2.5} 0.0" rpy="0 0 0"/>-->
+    <!--<origin xyz="-${src_box_w * 0.5 + src_box_h * 2.5} ${ty - src_box_w - src_box_h * 2.5} 0.0" rpy="0 0 0"/>-->
   <!--</joint>-->
   <!--<joint name="world_box_7_joint" type="fixed">-->
     <!--<parent link="world"/>-->
     <!--<child link="box_7_base"/>-->
-    <!--<origin xyz="${src_box_w * 0.5 - src_box_h * 2.5} ${ws_ysize - src_box_w - src_box_h * 0.5} ${tz}" rpy="0 0 0"/>-->
+    <!--<origin xyz="${src_box_w * 0.5 - src_box_h * 2.5} ${ty - src_box_w - src_box_h * 0.5} ${tz}" rpy="0 0 0"/>-->
   <!--</joint>-->
   <joint name="world_box_dst_joint" type="fixed">
     <parent link="world"/>
     <child link="box_dst_base"/>
-    <origin xyz="-${src_box_w * 1.0 + dst_box_h * 0.5 + src_box_h * 2.5} ${ws_ysize - src_box_w - src_box_h * 2.0 + dst_box_h * 0.5} 0.0" rpy="0 0 ${half_pi}"/>
+    <origin xyz="-${0.55 + dst_box_h * 0.5} ${0.05 + dst_box_w * 0.5} 0.0" rpy="0 0 ${half_pi}"/>
   </joint>
 </robot>

File: universal_robot/ur_description/urdf/ur5_joint_limited_robot.urdf.xacro (robot description, xacro)
@@ -22,5 +22,5 @@
     <parent link="table" />
     <child link = "base_link" />
-    <origin xyz="-0.105 0.09 0.0" rpy="0.0 0.0 1.57079632679" />
+    <origin xyz="-0.125 0.125 0.0" rpy="0.0 0.0 ${pi / 4.0}" />
   </joint>
   <joint name="ee_joint" type="fixed">

File: universal_robot/ur_description/urdf/ur5_robot.urdf.xacro (robot description, xacro)
@@ -16,5 +16,5 @@
     <parent link="table" />
     <child link = "base_link" />
-    <origin xyz="-0.105 0.09 0.0" rpy="0.0 0.0 1.57079632679" />
+    <origin xyz="-0.125 0.125 0.0" rpy="0.0 0.0 0.7853981633974483" />
   </joint>
   <joint name="ee_joint" type="fixed">
