Commit message: Update programs and params

File: universal_robot/ur_description/urdf/env/box.v2.urdf.xacro (robot description, xacro)
@@ -6,5 +6,5 @@
   <xacro:property name="src_box_w" value="0.43" />
   <xacro:property name="src_box_h" value="0.28" />
-  <xacro:property name="src_box_z" value="0.164" />
+  <xacro:property name="src_box_z" value="0.175" />
   <!-- Definitions of box destination dimensions  -->
   <xacro:property name="dst_box_w" value="0.33" />

File: universal_robot/ur_description/urdf/ur5_joint_limited_robot.urdf.xacro (robot description, xacro)
@@ -11,9 +11,13 @@
   <xacro:include filename="$(find ur_description)/urdf/actuator.urdf.xacro" />
   <!-- arm -->
+  <xacro:property name="shoulder_pan_min" value="-2.15050727526" />
+  <xacro:property name="shoulder_pan_max" value="-0.38351947466" />
+  <xacro:property name="elbow_joint_max" value="-0.735245529805" />
+  <xacro:property name="wrist_1_max" value="-0.316594425832" />
   <xacro:ur5_robot prefix="" joint_limited="true"
-    shoulder_pan_lower_limit="${-pi}" shoulder_pan_upper_limit="${pi}"
+    shoulder_pan_lower_limit="${shoulder_pan_min}" shoulder_pan_upper_limit="${shoulder_pan_max}"
     shoulder_lift_lower_limit="${-pi}" shoulder_lift_upper_limit="${pi}"
-    elbow_joint_lower_limit="${-pi}" elbow_joint_upper_limit="${pi}"
-    wrist_1_lower_limit="${-pi}" wrist_1_upper_limit="${pi}"
+    elbow_joint_lower_limit="${-pi}" elbow_joint_upper_limit="${elbow_joint_max}"
+    wrist_1_lower_limit="${-pi}" wrist_1_upper_limit="${wrist_1_max}"
     wrist_2_lower_limit="${-pi}" wrist_2_upper_limit="${pi}"
     wrist_3_lower_limit="${-pi}" wrist_3_upper_limit="${pi}"
