Commit message: Update srdf, link names etc and removed box 1 from the workspace

File: universal_robot/ur_description/urdf/actuator.urdf.xacro (robot description, xacro)
@@ -1,5 +1,5 @@
 ﻿<?xml version="1.0" encoding="UTF-8"?>
 <robot name="actuator" xmlns:xacro="http://ros.org/wiki/xacro">
-    <link name="base_plexi">
+    <link name="base_plexi_link">
         <visual>
             <origin xyz="0 0 0" rpy="0 0 0"/>
@@ -17,5 +17,5 @@
         </collision>
     </link>
-    <link name="base_plexi_2">
+    <link name="base_plexi_2_link">
         <visual>
             <origin xyz="0 0 0" rpy="0 0 0"/>
@@ -33,5 +33,5 @@
         </collision>
     </link>
-    <link name="venturi">
+    <link name="venturi_link">
         <origin xyz="0 0 0" rpy="0 0 0"/>
         <visual>
@@ -49,5 +49,5 @@
         </collision>
     </link>
-    <link name="ventouse">
+    <link name="suction_pad_link">
         <origin xyz="0 0 0" rpy="0 0 0"/>
         <visual>
@@ -65,17 +65,17 @@
         </collision>
     </link>
-    <joint name="base_plexi_to_base_plexi_2" type="fixed">
-        <parent link="base_plexi"/>
-        <child link="base_plexi_2"/>
+    <joint name="base_plexi_joint" type="fixed">
+        <parent link="base_plexi_link"/>
+        <child link="base_plexi_2_link"/>
         <origin xyz="0 0 0.008 "/>
     </joint>
-    <joint name="base_plexi_2_to_venturi" type="fixed">
-        <parent link="base_plexi_2"/>
-        <child link="venturi"/>
+    <joint name="base_plexi_2_joint" type="fixed">
+        <parent link="base_plexi_2_link"/>
+        <child link="venturi_link"/>
         <origin xyz="0 0 0.014 "/>
     </joint>
-    <joint name="adapteur_to_ventouse" type="fixed">
-        <parent link="venturi"/>
-        <child link="ventouse"/>
+    <joint name="venturi_joint" type="fixed">
+        <parent link="venturi_link"/>
+        <child link="suction_pad_link"/>
         <origin xyz="0.0 0.0 0.0225 "/>
     </joint>

File: universal_robot/ur_description/urdf/env/box.v2.urdf.xacro (robot description, xacro)
@@ -1,4 +1,4 @@
 ﻿<?xml version="1.0" encoding="UTF-8"?>
-<robot name="actuateur">
+<robot name="box">
   <link name="base">
     <visual>

File: universal_robot/ur_description/urdf/project_environment.urdf.xacro (robot description, xacro)
@@ -8,5 +8,5 @@
   <link name="world"/>
   <xacro:table name="table"/>
-  <xacro:box_source name="box_1"/>
+  <!--<xacro:box_source name="box_1"/>-->
   <xacro:box_source name="box_2"/>
   <xacro:box_source name="box_3"/>
@@ -21,9 +21,9 @@
     <origin xyz="-0.105 0.065 0.025" rpy="0 0 0"/>
   </joint>
-  <joint name="world_box_1_joint" type="fixed">
-    <parent link="world"/>
-    <child link="box_1"/>
-    <origin xyz="0.0 ${ws_ysize - bsw} ${bsz}" rpy="0 0 0"/>
-  </joint>
+  <!--<joint name="world_box_1_joint" type="fixed">-->
+    <!--<parent link="world"/>-->
+    <!--<child link="box_1"/>-->
+    <!--<origin xyz="0.0 ${ws_ysize - bsw} ${bsz}" rpy="0 0 0"/>-->
+  <!--</joint>-->
   <joint name="world_box_2_joint" type="fixed">
     <parent link="world"/>

File: universal_robot/ur_description/urdf/ur5_joint_limited_robot.urdf.xacro (robot description, xacro)
@@ -8,4 +8,6 @@
   <!-- ur5 -->
   <xacro:include filename="$(find ur_description)/urdf/ur5.urdf.xacro" />
+  <!-- actuator -->
+  <xacro:include filename="$(find ur_description)/urdf/actuator.urdf.xacro" />
   <!-- arm -->
   <xacro:ur5_robot prefix="" joint_limited="true"
@@ -22,3 +24,8 @@
     <origin xyz="-0.105 0.09 0.0" rpy="0.0 0.0 1.57079632679" />
   </joint>
+  <joint name="ee_joint" type="fixed">
+    <parent link="ee_link" />
+    <child link = "base_plexi_link" />
+    <origin xyz="0.004 0.0 0.0 " rpy="0.0 1.57079632679 0.0" />
+  </joint>
 </robot>

File: universal_robot/ur_description/urdf/ur5_robot.urdf.xacro (robot description, xacro)
@@ -17,8 +17,8 @@
     <origin xyz="-0.105 0.09 0.0" rpy="0.0 0.0 1.57079632679" />
   </joint>
-  <joint name="ee_link_table_base_plexi_joint" type="fixed">
+  <joint name="ee_joint" type="fixed">
     <parent link="ee_link" />
-    <child link = "base_plexi" />
-    <origin xyz="0.0 0.0 0.0" rpy="0.0 1.57079632679 0.0" />
+    <child link = "base_plexi_link" />
+    <origin xyz="0.004 0.0 0.0 " rpy="0.0 1.57079632679 0.0" />
   </joint>
 </robot>

Commit message: Update demo and all configs around

File: universal_robot/ur_description/urdf/actuator.urdf.xacro (robot description, xacro)
@@ -1,7 +1,8 @@
 ﻿<?xml version="1.0" encoding="UTF-8"?>
 <robot name="actuator" xmlns:xacro="http://ros.org/wiki/xacro">
+    <xacro:property name="half_pi" value="1.57079632679" />
     <link name="base_plexi_link">
         <visual>
-            <origin xyz="0 0 0" rpy="0 0 0"/>
+            <origin xyz="0 0 0" rpy="0 -${half_pi} 0"/>
             <geometry>
                 <cylinder length="0.008" radius="0.031"/>
@@ -12,4 +13,5 @@
         </visual>
         <collision>
+            <origin xyz="0 0 0" rpy="0 -${half_pi} 0"/>
             <geometry>
                 <cylinder length="0.008" radius="0.031"/>
@@ -19,5 +21,5 @@
     <link name="base_plexi_2_link">
         <visual>
-            <origin xyz="0 0 0" rpy="0 0 0"/>
+            <origin xyz="0 0 0" rpy="0 -${half_pi} 0"/>
             <geometry>
                 <cylinder length="0.008" radius="0.031"/>
@@ -28,4 +30,5 @@
         </visual>
         <collision>
+            <origin xyz="0 0 0" rpy="0 -${half_pi} 0"/>
             <geometry>
                 <cylinder length="0.008" radius="0.031"/>
@@ -34,6 +37,6 @@
     </link>
     <link name="venturi_link">
-        <origin xyz="0 0 0" rpy="0 0 0"/>
         <visual>
+            <origin xyz="0 0 0" rpy="0 -${half_pi} 0"/>
             <geometry>
                 <box size="0.038 0.038 .020"/>
@@ -44,4 +47,5 @@
         </visual>
         <collision>
+            <origin xyz="0 0 0" rpy="0 -${half_pi} 0"/>
             <geometry>
                 <box size="0.038 0.038 .020"/>
@@ -50,6 +54,6 @@
     </link>
     <link name="suction_pad_link">
-        <origin xyz="0 0 0" rpy="0 0 0"/>
         <visual>
+            <origin xyz="0 0 0" rpy="0 -${half_pi} 0"/>
             <geometry>
                 <cylinder length="0.025" radius="0.014"/>
@@ -60,4 +64,5 @@
         </visual>
         <collision>
+            <origin xyz="0 0 0" rpy="0 -${half_pi} 0"/>
             <geometry>
                 <cylinder length="0.025" radius="0.014"/>
@@ -68,15 +73,15 @@
         <parent link="base_plexi_link"/>
         <child link="base_plexi_2_link"/>
-        <origin xyz="0 0 0.008 "/>
+        <origin xyz="0.008 0 0 "/>
     </joint>
     <joint name="base_plexi_2_joint" type="fixed">
         <parent link="base_plexi_2_link"/>
         <child link="venturi_link"/>
-        <origin xyz="0 0 0.014 "/>
+        <origin xyz="0.014 0 0 "/>
     </joint>
     <joint name="venturi_joint" type="fixed">
         <parent link="venturi_link"/>
         <child link="suction_pad_link"/>
-        <origin xyz="0.0 0.0 0.0225 "/>
+        <origin xyz="0.0225 0.0 0.0 "/>
     </joint>
 </robot>

File: universal_robot/ur_description/urdf/ur5_joint_limited_robot.urdf.xacro (robot description, xacro)
@@ -27,5 +27,5 @@
     <parent link="ee_link" />
     <child link = "base_plexi_link" />
-    <origin xyz="0.004 0.0 0.0 " rpy="0.0 1.57079632679 0.0" />
+    <origin xyz="0.004 0.0 0.0 " rpy="1.57079632679 0.0 0.0" />
   </joint>
 </robot>

File: universal_robot/ur_description/urdf/ur5_robot.urdf.xacro (robot description, xacro)
@@ -2,4 +2,5 @@
 <robot xmlns:xacro="http://ros.org/wiki/xacro"
        name="ur5" >
+cd
   <!-- common stuff -->
   <xacro:include filename="$(find ur_description)/urdf/common.gazebo.xacro" />
@@ -20,5 +21,5 @@
     <parent link="ee_link" />
     <child link = "base_plexi_link" />
-    <origin xyz="0.004 0.0 0.0 " rpy="0.0 1.57079632679 0.0" />
+    <origin xyz="0.004 0.0 0.0 " rpy="1.57079632679 0.0 0.0" />
   </joint>
 </robot>
